File: RJ11Adapter/RJ11Adapter.sch (KiCad schematic (older format))
At the start: 3 parts, among them J1 RAIN_GAUGE, J2 WIND_RAIN, J3 WIND

Commit message: New A-2014-1-4-N-T-R Footprint
Parts:
- J1, J3: symbol KevinsLib:A-2014-1-4-N-T-R -> KevinLib:A-2014-1-4-N-T-R
Changed lines of the file:
@@
 $EndDescr
 $Comp
-L KevinsLib:A-2014-1-4-N-T-R J1
+L KevinLib:A-2014-1-4-N-T-R J1
 U 1 1 5F701278
 P 2950 2750
@@
 $EndComp
 $Comp
-L KevinsLib:A-2014-1-4-N-T-R J3
+L KevinLib:A-2014-1-4-N-T-R J3
 U 1 1 5F701C6E
 P 4850 2750
