File: WeatherSensors/WeatherStation.kicad_pcb (KiCad board)
At the start: 2 copper layers, 92.5 x 41 mm, 43 parts, among them J1 PROG_HEADER, J2 I2C_PORT, J3 LIGHT_HEADER, J4 WIND_RAIN, J5 PWR_HEADER, J6 BATTERY_HEADER, Q1 Q_NMOS_GSD, SW1 SW_EN, SW2 SW_I00, U1 ESP32-WROOM-32D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

Commit message: New A-2014-1-4-N-T-R Footprint
Changed lines of the file:
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@@
   )
   (setup
-    (last_trace_width 0.25)
+    (last_trace_width 0.254)
     (user_trace_width 0.1524)
     (user_trace_width 0.2)
@@
     (tags "capacitor handsolder")
     (attr smd)
-    (fp_text reference C2 (at 0 -1.65 90) (layer F.SilkS)
+    (fp_text reference C2 (at -0.1 1.6 90) (layer F.SilkS)
       (effects (font (size 1 1) (thickness 0.15)))
     )
@@
     (tags "capacitor handsolder")
     (attr smd)
-    (fp_text reference C3 (at 0 -1.65 90) (layer F.SilkS)
+    (fp_text reference C3 (at 0 1.2 90) (layer F.SilkS)
       (effects (font (size 1 1) (thickness 0.15)))
     )
@@
     (tags "capacitor handsolder")
     (attr smd)
-    (fp_text reference C8 (at 0 -1.65 90) (layer F.SilkS)
+    (fp_text reference C8 (at -2.9 -0.1 180) (layer F.SilkS)
       (effects (font (size 1 1) (thickness 0.15)))
     )
@@
     (descr "CP, Radial series, Radial, pin pitch=2.50mm, , diameter=5mm, Electrolytic Capacitor")
     (tags "CP Radial series Radial pin pitch 2.50mm  diameter 5mm Electrolytic Capacitor")
-    (fp_text reference C9 (at 1.25 -3.75 90) (layer F.SilkS)
+    (fp_text reference C9 (at -2.3 0.1 180) (layer F.SilkS)
       (effects (font (size 1 1) (thickness 0.15)))
     )
@@
     (descr "JST PH series connector, B4B-PH-K (http://www.jst-mfg.com/product/pdf/eng/ePH.pdf), generated with kicad-footprint-generator")
     (tags "connector JST PH side entry")
-    (fp_text reference J2 (at 3 -2.9) (layer F.SilkS)
+    (fp_text reference J2 (at -3.7 0) (layer F.SilkS)
       (effects (font (size 1 1) (thickness 0.15)))
     )
@@
     (descr "JST PH series connector, B6B-PH-K (http://www.jst-mfg.com/product/pdf/eng/ePH.pdf), generated with kicad-footprint-generator")
     (tags "connector JST PH side entry")
-    (fp_text reference J4 (at 5 -2.9) (layer F.SilkS)
+    (fp_text reference J4 (at -3.2 0.1) (layer F.SilkS)
       (effects (font (size 1 1) (thickness 0.15)))
     )
@@
     (descr "Through hole straight pin header, 1x05, 2.54mm pitch, single row")
     (tags "Through hole pin header THT 1x05 2.54mm single row")
-    (fp_text reference J5 (at 0 -2.33 90) (layer F.SilkS)
+    (fp_text reference J5 (at 0 -2.33 180) (layer F.SilkS)
       (effects (font (size 1 1) (thickness 0.15)))
     )
@@
     (descr "JST PH series connector, B2B-PH-K (http://www.jst-mfg.com/product/pdf/eng/ePH.pdf), generated with kicad-footprint-generator")
     (tags "connector JST PH side entry")
-    (fp_text reference J6 (at 1 1.6 90) (layer F.SilkS)
+    (fp_text reference J6 (at 5.1 0.3 180) (layer F.SilkS)
       (effects (font (size 1 1) (thickness 0.15)))
     )
@@
     (tags "resistor handsolder")
     (attr smd)
-    (fp_text reference R10 (at 0 -1.65 90) (layer F.SilkS)
-      (effects (font (size 1 1) (thickness 0.15)))
-    )
+    (fp_text reference R10 (at 0.1 -1.2 90) (layer F.SilkS)
+      (effects (font (size 1 1) (thickness 0.15)))
+    )
